Commit message: updated scale and visualization of accel_mag orientation rviz visualization

File: src/phone_description/urdf/phone.xacro (robot description, xacro)
@@ -13,10 +13,10 @@
     <collision name = "collision">
       <geometry>
-        <mesh filename = "package://phone_description/meshes/phone_new.dae"/>
+        <mesh filename = "package://phone_description/meshes/phone_new.dae" scale="100 100 100"/>
       </geometry>
     </collision>
     <visual name = "visual">
       <geometry>
-        <mesh filename = "package://phone_description/meshes/phone_new.dae"/>
+        <mesh filename = "package://phone_description/meshes/phone_new.dae" scale="100 100 100"/>
       </geometry>
     </visual>
